File: solenoid_driver/solenoid_driver.sch (KiCad schematic (older format))
At the start: 29 parts, among them J1 Conn_02x03_Odd_Even, J2 Conn_01x02, J3 Conn_01x02, J4 Conn_01x02, U1 FP6291, U2 ULN2003A, U3 TPS2553DBVR

Commit message: added version 1.0b with alternative inductor, because the inductor used by version 1.0 is low on stock. This variant has not been tested.
Parts:
- L1: footprint solenoid_driver_footprint_library:footprint_for_MWSA0503_HANDSOLD -> solenoid_driver_footprint_library:footprint_for_MWSA0402; LCSC C408410 -> C408337
Changed lines of the file:
@@
 F 0 "L1" H 8050 3990 50  0000 C CNN
 F 1 "4.7uH" H 8050 3899 50  0000 C CNN
-F 2 "solenoid_driver_footprint_library:footprint_for_MWSA0503_HANDSOLD" H 8050 3775 50  0001 C CNN
+F 2 "solenoid_driver_footprint_library:footprint_for_MWSA0402" H 8050 3775 50  0001 C CNN
 F 3 "https://datasheet.lcsc.com/szlcsc/1908262302_Sunlord-MWSA0503S-4R7MT_C408410.pdf" H 8050 3775 50  0001 C CNN
-F 4 "C408410" H 8050 3775 50  0001 C CNN "LCSC"
+F 4 " C408337" H 8050 3775 50  0001 C CNN "LCSC"
 	1    8050 3775
 	1    0    0    -1

Commit message: Use handsoldered footprint, add 3d model
Parts:
- L1: footprint solenoid_driver_footprint_library:footprint_for_MWSA0402 -> solenoid_driver_footprint_library:footprint_for_MWSA0402_HANDSOLD
Changed lines of the file:
@@
 F 0 "L1" H 8050 3990 50  0000 C CNN
 F 1 "4.7uH" H 8050 3899 50  0000 C CNN
-F 2 "solenoid_driver_footprint_library:footprint_for_MWSA0402" H 8050 3775 50  0001 C CNN
+F 2 "solenoid_driver_footprint_library:footprint_for_MWSA0402_HANDSOLD" H 8050 3775 50  0001 C CNN
 F 3 "https://datasheet.lcsc.com/szlcsc/1908262302_Sunlord-MWSA0503S-4R7MT_C408410.pdf" H 8050 3775 50  0001 C CNN
 F 4 " C408337" H 8050 3775 50  0001 C CNN "LCSC"

Commit message: Updated 100k resistor and 22uF capacitor part references
Parts:
- C5, C6: LCSC C45783 -> C602037
- R1, R2, R5, R8: LCSC C17407 -> C149504
Changed lines of the file:
@@
 F 2 "Resistor_SMD:R_0805_2012Metric_Pad1.15x1.40mm_HandSolder" V 4955 3500 50  0001 C CNN
 F 3 "~" H 5025 3500 50  0001 C CNN
-F 4 "C17407" H 5025 3500 50  0001 C CNN "LCSC"
+F 4 "C149504" H 5025 3500 50  0001 C CNN "LCSC"
 	1    5025 3500
 	1    0    0    -1
@@
 F 2 "Resistor_SMD:R_0805_2012Metric_Pad1.15x1.40mm_HandSolder" V 9030 3375 50  0001 C CNN
 F 3 "~" H 9100 3375 50  0001 C CNN
-F 4 "C17407" H 9100 3375 50  0001 C CNN "LCSC"
+F 4 "C149504" H 9100 3375 50  0001 C CNN "LCSC"
 	1    9100 3375
 	1    0    0    -1
@@
 F 2 "Capacitor_SMD:C_0805_2012Metric_Pad1.15x1.40mm_HandSolder" H 6813 2950 50  0001 C CNN
 F 3 "~" H 6775 3100 50  0001 C CNN
-F 4 "C45783" H 6775 3100 50  0001 C CNN "LCSC"
+F 4 "C602037" H 6775 3100 50  0001 C CNN "LCSC"
 	1    6775 3100
 	1    0    0    -1
@@
 F 2 "Capacitor_SMD:C_0805_2012Metric_Pad1.15x1.40mm_HandSolder" H 9488 3050 50  0001 C CNN
 F 3 "~" H 9450 3200 50  0001 C CNN
-F 4 "C45783" H 9450 3200 50  0001 C CNN "LCSC"
+F 4 "C602037" H 9450 3200 50  0001 C CNN "LCSC"
 	1    9450 3200
 	1    0    0    -1
@@
 F 2 "Resistor_SMD:R_0805_2012Metric_Pad1.15x1.40mm_HandSolder" V 7630 3250 50  0001 C CNN
 F 3 "~" H 7700 3250 50  0001 C CNN
-F 4 "C17407" H 7700 3250 50  0001 C CNN "LCSC"
+F 4 "C149504" H 7700 3250 50  0001 C CNN "LCSC"
 	1    7700 3250
 	1    0    0    -1
@@
 F 2 "Resistor_SMD:R_0805_2012Metric_Pad1.15x1.40mm_HandSolder" V 6305 2550 50  0001 C CNN
 F 3 "~" H 6375 2550 50  0001 C CNN
-F 4 "C17407" H 6375 2550 50  0001 C CNN "LCSC"
+F 4 "C149504" H 6375 2550 50  0001 C CNN "LCSC"
 	1    6375 2550
 	1    0    0    -1
